File: TABv1.kicad_pcb (KiCad board)
At the start: 4 copper layers, 90 x 45 mm, 127 parts, among them IC1 TPS630702RNMR, J1 USB_C_Receptacle_USB2.0_16P, J11 Conn_UART_1, J15 DB141R-2.54-8P-GN, J2 Conn_02x03_Row_Letter_Last, J3 Conn_02x03_Row_Letter_Last, J4 Conn_Coaxial, J5 Conn_02x06_Counter_Clockwise, J6 SWD, J7 503398-1892, J8 1053141104, Q1 MJD44H11T4G, Q10 PJM09P30DF, Q11 PJM09P30DF, Q12 PJM09P30DF, Q13 PJM09P30DF, Q2 NMOS, Q5 NMOS, Q6 NMOS, Q7 NMOS, Q8 NMOS, Q9 NMOS, SW1 BOOTSEL, SW2 RESET, U1 RP2350B-QFN80, U10 RAK3172, U11 LPS22DF, U2 W25Q128JVS, U4 LSM6DSO32TR, U6 LT3092xST, U7 LSM6DSO32TR, U8 LIS2MDL, U9 TESEO-LIV4F, Y1 12MHz

Commit message: small_changes
Parts:
- moved R20 10.0 mm to (139.1, 44.1)
- moved C21 3.01 mm to (148.0, 40.4)
- moved R21 1.75 mm to (149.1, 44.3)
- moved R22 1.71 mm to (147.4, 44.3)
- moved R27 0.86 mm to (145.9, 71.1)
- moved Q12 0.71 mm to (150.7, 68.3)
- moved Q8 0.71 mm to (146.5, 68.2)
- moved R33 0.71 mm to (146.0, 65.5)
- moved R34 0.67 mm to (150.4, 64.6)
- moved R17 0.66 mm to (148.7, 64.6)
- moved R28 0.66 mm to (145.9, 72.8)
- moved R32 0.61 mm to (146.0, 63.8)
- moved R12 0.57 mm to (148.9, 71.9)
- moved R14 0.56 mm to (150.6, 71.9)
- moved Q10 0.51 mm to (150.8, 75.4)
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Routing:
- net /PYRO_FIRE_3: track 46.1 -> 13.3 mm
- net /Pyro/PYRO3: track 4.04 -> 0.00 mm
- net /Pyro/PYRO2: track 18.5 -> 14.5 mm, vias 1 -> 0
- net GND: track 102.4 -> 99.3 mm
- net Net-(Q12-G): track 4.45 -> 2.45 mm
- net /Pyro/PYRO_HIGH: track 13.0 -> 14.2 mm
- net Net-(Q6-G): track 3.50 -> 4.29 mm
- net /Pyro/PYRO1: track 7.71 -> 8.39 mm
