File: TABv1.kicad_pcb (KiCad board)
At the start: 4 copper layers, 90 x 45 mm, 127 parts, among them IC1 TPS630702RNMR, J1 USB_C_Receptacle_USB2.0_16P, J10 Conn_02x03_Odd_Even, J11 Conn_UART_1, J15 DB141R-2.54-8P-GN, J4 Conn_Coaxial, J5 Conn_02x06_Counter_Clockwise, J6 SWD, J7 503398-1892, J8 1053141104, J9 Conn_02x03_Odd_Even, Q1 MJD44H11T4G, Q10 PJM09P30DF, Q11 PJM09P30DF, Q12 PJM09P30DF, Q13 PJM09P30DF, Q2 NMOS, Q5 NMOS, Q6 NMOS, Q7 NMOS, Q8 NMOS, Q9 NMOS, SW1 BOOTSEL, SW2 RESET, U1 RP2350B-QFN80, U10 RAK3172, U11 LPS22DF, U2 W25Q128JVS, U4 LSM6DSO32TR, U6 LT3092xST, U7 LSM6DSO32TR, U8 LIS2MDL, U9 TESEO-LIV4F, Y1 12MHz

Commit message: Changes 11/12
Parts:
- C12, C15: moved to B.Cu
- moved C11 3.26 mm to (90.5, 68.2), turned to 0 degrees
- moved C9 3.20 mm to (90.5, 66.7), turned to 0 degrees
- moved C15 1.35 mm to (85.8, 57.3)
- moved C12 1.25 mm to (85.8, 55.7)
- moved C10 1.05 mm to (86.0, 61.9)
Connections:
- J10 pad 1: /PWM4 -> /PWM2
- J10 pad 2: /PWM3 -> /PWM1
- J9 pad 1: /PWM2 -> /PWM4
- J9 pad 2: /PWM1 -> /PWM3
- U1 pad 42: unconnected-(U1-GPIO33-Pad42) -> /BUZZ
- U1 pad 56: /L_BLUE -> unconnected-(U1-GPIO45_ADC5-Pad56)
- U1 pad 57: /BUZZ -> unconnected-(U1-GPIO46_ADC6-Pad57)
Routing:
- net /PWM1: track 0.00 -> 82.4 mm, vias 0 -> 2
- net /PWM2: track 0.00 -> 78.8 mm, vias 0 -> 2
- net /PWM3: track 0.00 -> 76.8 mm, vias 0 -> 2
- net /PWM4: track 0.00 -> 75.2 mm, vias 0 -> 2
- net /SD_DAT0: track 0.00 -> 51.3 mm, vias 0 -> 2
- net /SD_CLK: track 48.2 -> 12.0 mm, vias 2 -> 1
- net /XIN: track 2.36 -> 24.8 mm
- net /SD0: track 4.71 -> 22.0 mm, vias 1 -> 2
- net /BARO_CS: track 10.5 -> 24.2 mm
- net /L_BLUE: track 29.9 -> 21.5 mm
- net /SD_DAT3: track 30.4 -> 38.3 mm
- net GND: track 167.2 -> 159.4 mm, vias 64 -> 65
- net /RX_GPS: track 60.7 -> 68.2 mm
- net /SD_DAT2: track 30.9 -> 35.2 mm
- net /SD_CMD: track 28.2 -> 32.1 mm
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
Commit message: Changes
Routing:
- net /IMU45_CS: track 22.1 -> 24.9 mm
- net GND: track 159.4 -> 161.6 mm, vias 65 -> 66
- net /PWM2: track 78.8 -> 80.6 mm
- net /PWM3: track 76.8 -> 78.5 mm
- net /PWM4: track 75.2 -> 74.1 mm
- net /SD_DAT3: track 38.3 -> 37.5 mm
- net /SD_detect: track 43.9 -> 44.5 mm
- net +3V3: track 126.1 -> 126.7 mm
- net /PWM1: track 82.4 -> 83.0 mm

Commit message: changes sat 13/12/25
Parts:
- Q2, R10, R11: moved to B.Cu
- moved LS1 45.2 mm to (127.7, 38.7), turned to 0 degrees
- moved Q2 36.0 mm to (118.8, 36.8), turned to 180 degrees
- moved R11 35.0 mm to (119.5, 42.0), turned to -90 degrees
- moved R10 33.0 mm to (117.5, 42.0)
- moved C12 1.77 mm to (84.5, 54.5)
- moved C15 1.77 mm to (84.5, 56.1)
- moved R40 1.53 mm to (112.2, 48.5)
Connections:
- J5 pad 11: /GPIO28 -> /PWM1
- J5 pad 5: /GPIO21 -> /PWM4
- J5 pad 7: /GPIO22 -> /PWM3
- J5 pad 9: /GPIO23 -> /PWM2
Routing:
- net /SD_DAT1: track 3.41 -> 53.7 mm, vias 1 -> 2
- net /BUZZ: track 0.00 -> 40.2 mm, vias 0 -> 3
- net /SD_CLK: track 12.0 -> 47.9 mm, vias 1 -> 2
- net +3V3: track 126.7 -> 157.9 mm, vias 30 -> 34
- net /PWM3: track 78.5 -> 104.8 mm
- net Net-(J11-Pin_2): track 0.00 -> 25.6 mm, vias 0 -> 2
- net Net-(J11-Pin_3): track 0.00 -> 24.9 mm, vias 0 -> 2
- net /PWM1: track 83.0 -> 107.8 mm
- net /PWM4: track 74.1 -> 98.7 mm
- net /PWM2: track 80.6 -> 104.3 mm
- net /SD3: track 4.70 -> 22.5 mm, vias 1 -> 3
- net /SPI1.RX: track 56.9 -> 46.2 mm
- net Net-(Q2-D): track 0.00 -> 4.75 mm
- net Net-(Q2-G): track 0.00 -> 4.30 mm
- net GND: track 161.6 -> 165.6 mm, vias 66 -> 70
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
Commit message: small
Parts:
- moved J11 0.20 mm to (89.2, 36.8)
Routing:
- net /GPIO43: track 0.00 -> 28.6 mm, vias 0 -> 1
- net GND: track 165.6 -> 169.4 mm, vias 70 -> 72
- net +3V3: track 157.9 -> 159.6 mm, vias 34 -> 35
- net /SD_CMD: track 33.5 -> 32.4 mm
- net VUSB: track 86.9 -> 85.9 mm
- net /SD_detect: track 45.7 -> 46.3 mm

Commit message: Collegamenti ultimati
Routing:
- net /GPIO41: track 0.00 -> 31.5 mm, vias 0 -> 2
- net /GPIO42: track 0.00 -> 31.3 mm, vias 0 -> 2
- net /GPIO44: track 0.00 -> 30.6 mm, vias 0 -> 1
- net /GPIO43: track 28.6 -> 31.7 mm, vias 1 -> 2
- net /PWM3: track 105.1 -> 103.3 mm
- net /SD3: track 22.9 -> 24.3 mm, vias 3 -> 4
- net Net-(J11-Pin_2): track 25.4 -> 24.3 mm
- net /PWM4: track 98.5 -> 97.7 mm
- net SYNC: track 6.26 -> 6.86 mm
- net +1V1: track 29.2 -> 29.5 mm, vias 4 -> 3

Commit message: .
Routing:
- net /GPIO20: track 0.00 -> 63.7 mm, vias 0 -> 2
- net GND: track 169.0 -> 172.2 mm, vias 72 -> 74
- net Net-(J7-DAT0): track 13.9 -> 14.5 mm

Commit message: Modifiche 18/12
Parts:
- moved J4 0.12 mm to (72.8, 64.4)

Commit message: changes 18/12
Parts:
- added G***: LOGO, LOGO, F.Cu at (117.7, 60.9)
- moved C20 0.78 mm to (144.5, 42.0)
- moved R33 0.31 mm to (145.8, 65.4)
- moved R32 0.28 mm to (145.8, 63.7)
- moved R35 0.27 mm to (145.6, 56.3)
- moved R36 0.27 mm to (145.6, 58.0)
Routing:
- net +1V1: track 29.5 -> 28.3 mm, vias 3 -> 2
- net Net-(IC1-VAUX): track 2.96 -> 3.72 mm
Other:
- outline, holes or cut-outs redrawn
- board text added: "CERERE"
- board text added: "REV 1.0"
