File: TABv1.kicad_sch (KiCad schematic)
At the start: 41 parts, among them J10 Conn_UART_HOST, J11 Conn_UART_1, J12 Conn_UART_0, J13 Conn_ADC, J2 Conn_02x03_Row_Letter_Last, J3 Conn_02x03_Row_Letter_Last, J6 SWD, J8 Conn_SPI1, J9 Conn_SPI0, Q2 NMOS, SW2 RESET, U1 RP2350B-QFN80, Y1 12MHz

Commit message: Update TABv1.kicad_sch
Parts:
- H1, H2, H3, H4: footprint MountingHole:MountingHole_2.2mm_M2 -> MountingHole:MountingHole_3.2mm_M3
Changed lines of the file:
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@@
 			)
 		)
-		(property "Footprint" "MountingHole:MountingHole_2.2mm_M2"
+		(property "Footprint" "MountingHole:MountingHole_3.2mm_M3"
 			(at 365.76 156.21 0)
 			(effects
@@
 			)
 		)
-		(property "Footprint" "MountingHole:MountingHole_2.2mm_M2"
+		(property "Footprint" "MountingHole:MountingHole_3.2mm_M3"
 			(at 365.76 149.86 0)
 			(effects
@@
 			)
 		)
-		(property "Footprint" "MountingHole:MountingHole_2.2mm_M2"
+		(property "Footprint" "MountingHole:MountingHole_3.2mm_M3"
 			(at 365.76 143.51 0)
 			(effects
@@
 			)
 		)
-		(property "Footprint" "MountingHole:MountingHole_2.2mm_M2"
+		(property "Footprint" "MountingHole:MountingHole_3.2mm_M3"
 			(at 365.76 162.56 0)
 			(effects

Commit message: fix
Parts:
- removed J10: Conn_UART_HOST, Connector_PinHeader_2.54mm:PinHeader_1x02_P2.54mm_Vertical, symbol Connector:Conn_01x02_Pin
- removed J12: Conn_UART_0, Connector_PinHeader_2.54mm:PinHeader_1x02_P2.54mm_Vertical, symbol Connector:Conn_01x02_Pin
Connections:
- net RX_GPS: now also U1.16 (GPIO16)
- net SCL_RADIO: now also U1.78 (GPIO1)
- net SDA_RADIO: now also U1.77 (GPIO0)
- net TX_GPS: now also U1.17 (GPIO17)
Changed lines of the file:
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@@
 	(wire
 		(pts
-			(xy 147.32 129.54) (xy 167.64 129.54)
+			(xy 147.32 129.54) (xy 182.88 129.54)
 		)
 		(stroke
@@
 	(wire
 		(pts
-			(xy 147.32 132.08) (xy 167.64 132.08)
+			(xy 147.32 132.08) (xy 182.88 132.08)
 		)
 		(stroke
@@
 	(wire
 		(pts
-			(xy 172.72 132.08) (xy 182.88 132.08)
-		)
-		(stroke
-			(width 0)
-			(type default)
-		)
-	)
-	(wire
-		(pts
 			(xy 217.17 123.19) (xy 232.41 123.19)
 		)
@@
 	(wire
 		(pts
-			(xy 172.72 129.54) (xy 182.88 129.54)
-		)
-		(stroke
-			(width 0)
-			(type default)
-		)
-	)
-	(wire
-		(pts
 			(xy 353.822 193.04) (xy 353.822 194.31)
 		)
@@
 	(wire
 		(pts
-			(xy 147.32 88.9) (xy 166.37 88.9)
+			(xy 147.32 88.9) (xy 173.99 88.9)
 		)
 		(stroke
@@
 	(wire
 		(pts
-			(xy 147.32 91.44) (xy 166.37 91.44)
+			(xy 147.32 91.44) (xy 173.99 91.44)
 		)
 		(stroke
@@
 	(wire
 		(pts
-			(xy 171.45 88.9) (xy 173.99 88.9)
-		)
-		(stroke
-			(width 0)
-			(type default)
-		)
-	)
-	(wire
-		(pts
 			(xy 342.9 87.63) (xy 345.44 87.63)
 		)
@@
 	(wire
 		(pts
-			(xy 171.45 91.44) (xy 173.99 91.44)
-		)
-		(stroke
-			(width 0)
-			(type default)
-		)
-	)
-	(wire
-		(pts
 			(xy 147.32 109.22) (xy 167.64 109.22)
 		)
@@
 	)
 	(symbol
-		(lib_id "Connector:Conn_01x02_Pin")
-		(at 172.72 132.08 180)
-		(unit 1)
-		(exclude_from_sim no)
-		(in_bom yes)
-		(on_board yes)
-		(dnp no)
-		(property "Reference" "J12"
-			(at 170.688 127 0)
-			(effects
-				(font
-					(size 1.27 1.27)
-				)
-				(justify right)
-			)
-		)
-		(property "Value" "Conn_UART_0"
-			(at 170.688 133.858 0)
-			(effects
-				(font
-					(size 1.27 1.27)
-				)
-				(justify right)
-			)
-		)
-		(property "Footprint" "Connector_PinHeader_2.54mm:PinHeader_1x02_P2.54mm_Vertical"
-			(at 172.72 132.08 0)
-			(effects
-				(font
-					(size 1.27 1.27)
-				)
-				(hide yes)
-			)
-		)
-		(property "Datasheet" "~"
-			(at 172.72 132.08 0)
-			(effects
-				(font
-					(size 1.27 1.27)
-				)
-				(hide yes)
-			)
-		)
-		(property "Description" "Generic connector, single row, 01x02, script generated"
-			(at 172.72 132.08 0)
-			(effects
-				(font
-					(size 1.27 1.27)
-				)
-				(hide yes)
-			)
-		)
-		(pin "1"
-		)
-		(pin "2"
-		)
-		(instances
-			(project "cockatiel"
-				(path "/105f6e80-8e20-4d56-8eb3-6fa826818670"
-					(reference "J12")
-					(unit 1)
-				)
-			)
-		)
-	)
-	(symbol
 		(lib_id "Connector:Conn_01x04_Pin")
 		(at 171.45 154.94 180)
@@
 					(unit 1)
 				)
-			)
-		)
-	)
-	(symbol
-		(lib_id "Connector:Conn_01x02_Pin")
-		(at 171.45 91.44 180)
-		(unit 1)
-		(exclude_from_sim no)
-		(in_bom yes)
-		(on_board yes)
-		(dnp no)
-		(property "Reference" "J10"
-			(at 169.672 87.122 0)
-			(effects
-				(font
-					(size 1.27 1.27)
-				)
-				(justify right)
-			)
-		)
-		(property "Value" "Conn_UART_HOST"
-			(at 168.402 93.218 0)
-			(effects
-				(font
-					(size 1.27 1.27)
-				)
-				(justify right)
-			)
-		)
-		(property "Footprint" "Connector_PinHeader_2.54mm:PinHeader_1x02_P2.54mm_Vertical"
-			(at 171.45 91.44 0)
-			(effects
-				(font
-					(size 1.27 1.27)
-				)
-				(hide yes)
-			)
-		)
-		(property "Datasheet" "~"
-			(at 171.45 91.44 0)
-			(effects
-				(font
-					(size 1.27 1.27)
-				)
-				(hide yes)
-			)
-		)
-		(property "Description" "Generic connector, single row, 01x02, script generated"
-			(at 171.45 91.44 0)
-			(effects
-				(font
-					(size 1.27 1.27)
-				)
-				(hide yes)
-			)
-		)
-		(pin "1"
-		)
-		(pin "2"
-		)
-		(instances
-			(project ""
-				(path "/105f6e80-8e20-4d56-8eb3-6fa826818670"
-					(reference "J10")
-					(unit 1)
-				)

Commit message: fix continuo
Parts:
- J11: footprint Connector_PinHeader_2.54mm:PinHeader_1x02_P2.54mm_Vertical -> Connector_JST:JST_XH_S2B-XH-A-1_1x02_P2.50mm_Horizontal
Changed lines of the file:
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@@
 			)
 		)
-		(property "Footprint" "Connector_PinHeader_2.54mm:PinHeader_1x02_P2.54mm_Vertical"
+		(property "Footprint" "Connector_JST:JST_XH_S2B-XH-A-1_1x02_P2.50mm_Horizontal"
 			(at 172.72 111.76 0)
 			(effects

Commit message: upload routing con rotellini
Parts:
- removed J13: Conn_ADC, Connector_PinHeader_2.54mm:PinHeader_1x04_P2.54mm_Vertical, symbol Connector:Conn_01x04_Pin
- removed J8: Conn_SPI1, Connector_PinHeader_2.54mm:PinHeader_1x04_P2.54mm_Vertical, symbol Connector:Conn_01x04_Pin
- added J5: Conn_02x06_Counter_Clockwise, Connector_PinHeader_2.54mm:PinHeader_2x06_P2.54mm_Vertical, symbol Connector_Generic:Conn_02x06_Odd_Even
- J11: footprint Connector_JST:JST_XH_S2B-XH-A-1_1x02_P2.50mm_Horizontal -> Connector_JST:JST_XH_B3B-XH-AM_1x03_P2.50mm_Vertical; symbol Connector:Conn_01x02_Pin -> Connector:Conn_01x03_Pin
Connections:
- net +3V3: now also J5.2 (Pin_2)
- net GND: now also J11.1 (Pin_1), J5.1 (Pin_1), J5.12 (Pin_12)
- net L_RED: no longer U1.36 (GPIO28)
- net at U1.7 (GPIO9): now also J11.2 (Pin_2); no longer J11.1 (Pin_1)
- net at U1.6 (GPIO8): now also J11.3 (Pin_3); no longer J11.2 (Pin_2)
- net GPIO27: now reaches U1.28 (GPIO27)
- net GPIO27: now also J5.9 (Pin_9)
- net GPIO26: now reaches U1.27 (GPIO26)
- net GPIO26: now also J5.7 (Pin_7)
- net GPIO25: now reaches U1.26 (GPIO25)
- net GPIO25: now also J5.5 (Pin_5)
- net GPIO24: now reaches U1.25 (GPIO24)
- net GPIO24: now also J5.3 (Pin_3)
- net GPIO41: now reaches U1.52 (GPIO41_ADC1)
- net GPIO41: now also J5.4 (Pin_4)
- net GPIO42: now reaches U1.53 (GPIO42_ADC2)
- net GPIO42: now also J5.6 (Pin_6)
- net GPIO43: now reaches U1.54 (GPIO43_ADC3)
- net GPIO43: now also J5.8 (Pin_8)
- net GPIO44: now reaches U1.55 (GPIO44_ADC4)
- net GPIO44: now also J5.10 (Pin_10)
- new net GPIO28: J5.11 (Pin_11), U1.36 (GPIO28)

Commit message: Changes meeting 03/12
Parts:
- removed J9: Conn_SPI0, Connector_PinHeader_2.54mm:PinHeader_1x04_P2.54mm_Vertical, symbol Connector:Conn_01x04_Pin
Connections:
- net PWM1: now also U1.25 (GPIO24); no longer U1.20 (GPIO20)
- net PWM2: now also U1.26 (GPIO25); no longer U1.21 (GPIO21)
- net PWM3: now also U1.27 (GPIO26); no longer U1.22 (GPIO22)
- net PWM4: now also U1.28 (GPIO27); no longer U1.23 (GPIO23)
- net BATT_SENSE: now reaches U1.58 (GPIO47_ADC7)
- net GPIO24 renamed GPIO20
- net GPIO20: now also U1.20 (GPIO20); no longer U1.25 (GPIO24)
- net GPIO25 renamed GPIO21
- net GPIO21: now also U1.21 (GPIO21); no longer U1.26 (GPIO25)
- net GPIO26 renamed GPIO22
- net GPIO22: now also U1.22 (GPIO22); no longer U1.27 (GPIO26)
- net GPIO27 renamed GPIO23
- net GPIO23: now also U1.23 (GPIO23); no longer U1.28 (GPIO27)
- no-connect marks 1 -> 0
Other:
- sheet Power ports: added BATT_SENSE; removed none
Changed lines of the file:
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@@
 		(color 0 0 0 0)
 	)
-	(no_connect
-		(at 147.32 210.82)
-	)
 	(bus_entry
 		(at 55.88 107.95)
@@
 		)
 	)
+	(wire
+		(pts
+			(xy 166.37 210.82) (xy 147.32 210.82)
+		)
+		(stroke
+			(width 0)
+			(type default)
+		)
+	)
 	(polyline
 		(pts
@@
 		)
 	)
+	(label "PWM4"
+		(at 166.37 157.48 0)
+		(effects
+			(font
+				(size 1.27 1.27)
+			)
+			(justify left bottom)
+		)
+	)
 	(label "IMU_INT2"
 		(at 166.37 175.26 180)
@@
 		)
 	)
-	(label "PWM2"
-		(at 177.8 142.24 0)
-		(effects
-			(font
-				(size 1.27 1.27)
-			)
-			(justify left bottom)
-		)
-	)
 	(label "XOUT"
 		(at 72.39 129.54 0)
@@
 		)
 	)
-	(label "GPIO27"
+	(label "GPIO23"
 		(at 207.01 205.74 180)
 		(effects
@@
 		)
 	)
-	(label "GPIO24"
-		(at 166.37 149.86 0)
+	(label "SCLK"
+		(at 57.15 114.3 0)
 		(effects
 			(font
@@
 		)
 	)
-	(label "SCLK"
-		(at 57.15 114.3 0)
+	(label "PWM1"
+		(at 166.37 149.86 0)
 		(effects
 			(font
@@
 		)
 	)
-	(label "GPIO24"
+	(label "GPIO20"
 		(at 207.01 198.12 180)
 		(effects
@@
 		)
 	)
+	(label "GPIO20"
+		(at 190.5 139.7 0)
+		(effects
+			(font
+				(size 1.27 1.27)
+			)
+			(justify left bottom)
+		)
+	)
 	(label "FB"
 		(at 57.15 87.63 0)
@@
 		)
 	)
+	(label "PWM2"
+		(at 166.37 152.4 0)
+		(effects
+			(font
+				(size 1.27 1.27)
+			)
+			(justify left bottom)
+		)
+	)
 	(label "SCL_RADIO"
 		(at 173.99 91.44 0)
@@
 		)
 	)
+	(label "BATT_SENSE"
+		(at 166.37 210.82 0)
+		(effects
+			(font
+				(size 1.27 1.27)
+			)
+			(justify left bottom)
+		)
+	)
 	(label "BARO_INT"
 		(at 217.17 107.95 0)
@@
 		)
 	)
-	(label "PWM1"
-		(at 177.8 139.7 0)
+	(label "GPIO22"
+		(at 190.5 144.78 0)
 		(effects
 			(font
@@
 		)
 	)
-	(label "GPIO26"
-		(at 166.37 154.94 0)
+	(label "SD2"
+		(at 57.15 107.95 0)
 		(effects
 			(font
@@
 		)
 	)
-	(label "SD2"
-		(at 57.15 107.95 0)
+	(label "LX"
+		(at 57.15 90.17 0)
 		(effects
 			(font
@@
 		)
 	)
-	(label "LX"
-		(at 57.15 90.17 0)
+	(label "GPIO21"
+		(at 190.5 142.24 0)
 		(effects
 			(font
@@
 		)
 	)
-	(label "GPIO25"
-		(at 166.37 152.4 0)
-		(effects
-			(font
-				(size 1.27 1.27)
-			)
-			(justify left bottom)
-		)
-	)
 	(label "SD0"
 		(at 57.15 102.87 0)
@@
 		)
 	)
-	(label "BARO_CS"
-		(at 166.37 165.1 180)
+	(label "GPIO23"
+		(at 190.5 147.32 0)
 		(effects
 			(font
 				(size 1.27 1.27)
 			)
-			(justify right bottom)
+			(justify left bottom)
 		)
 	)
-	(label "L_GREEN"
-		(at 166.37 162.56 0)
+	(label "BARO_CS"
+		(at 166.37 165.1 180)
 		(effects
 			(font
 				(size 1.27 1.27)
 			)
-			(justify left bottom)
+			(justify right bottom)
 		)
 	)
-	(label "PWM4"
-		(at 177.8 147.32 0)
+	(label "L_GREEN"
+		(at 166.37 162.56 0)
 		(effects
 			(font
@@
 		)
 	)
-	(label "PWM3"
-		(at 177.8 144.78 0)
-		(effects
-			(font
-				(size 1.27 1.27)
-			)
-			(justify left bottom)
-		)
-	)
 	(label "SD_DAT0"
 		(at 166.37 99.06 180)
@@
 		)
 	)
+	(label "BATT_SENSE"
+		(at 232.41 41.91 180)
+		(effects
+			(font
+				(size 1.27 1.27)
+			)
+			(justify right bottom)
+		)
+	)
 	(label "L_RED"
 		(at 352.806 193.04 180)
@@
 		)
 	)
-	(label "GPIO25"
+	(label "GPIO21"
 		(at 207.01 200.66 180)
 		(effects
@@
 		)
 	)
-	(label "GPIO26"
+	(label "GPIO22"
 		(at 207.01 203.2 180)
 		(effects
@@
 		)
 	)
-	(label "GPIO27"
-		(at 166.37 157.48 0)
-		(effects
-			(font
-				(size 1.27 1.27)
-			)
-			(justify left bottom)
-		)
-	)
 	(label "PYRO_FIRE_3"
 		(at 166.37 185.42 180)
@@
 		)
 	)
+	(label "PWM3"
+		(at 166.37 154.94 0)
+		(effects
+			(font
+				(size 1.27 1.27)
+			)
+			(justify left bottom)
+		)
+	)
 	(label "PYRO_ENABLE"
 		(at 246.38 156.21 0)
@@
 	)
 	(symbol
-		(lib_id "Connector:Conn_01x04_Pin")
-		(at 195.58 144.78 180)
-		(unit 1)
-		(exclude_from_sim no)
-		(in_bom yes)
-		(on_board yes)
-		(dnp no)
-		(property "Reference" "J9"
-			(at 196.85 142.2399 0)
-			(effects
-				(font
-					(size 1.27 1.27)
-				)
-				(justify right)
-			)
-		)
-		(property "Value" "Conn_SPI0"
-			(at 201.168 144.272 0)
-			(effects
-				(font
-					(size 1.27 1.27)
-				)
-				(justify right)
-			)
-		)
-		(property "Footprint" "Connector_PinHeader_2.54mm:PinHeader_1x04_P2.54mm_Vertical"
-			(at 195.58 144.78 0)
-			(effects
-				(font
-					(size 1.27 1.27)
-				)
-				(hide yes)
-			)
-		)
-		(property "Datasheet" "~"
-			(at 195.58 144.78 0)
-			(effects
-				(font
-					(size 1.27 1.27)
-				)
-				(hide yes)
-			)
-		)
-		(property "Description" "Generic connector, single row, 01x04, script generated"
-			(at 195.58 144.78 0)
-			(effects
-				(font
-					(size 1.27 1.27)
-				)
-				(hide yes)
-			)
-		)
-		(pin "2"
-		)
-		(pin "4"
-		)
-		(pin "3"
-		)
-		(pin "1"
-		)
-		(instances
-			(project "cockatiel"
-				(path "/105f6e80-8e20-4d56-8eb3-6fa826818670"
-					(reference "J9")
-					(unit 1)
-				)
-			)
-		)
-	)
-	(symbol
 		(lib_id "power:+3V3")
 		(at 137.16 60.96 0)
@@
 			(effects
 				(font
+					(size 1.27 1.27)
+				)
+				(justify left)
+			)
+		)
+		(pin "BATT_SENSE" input
+			(at 232.41 41.91 180)
+			(effects
+				(font

Commit message: Routing Changes
Parts:
- removed J2, J3: Conn_02x03_Row_Letter_Last, Connector_PinHeader_2.54mm:PinHeader_2x03_P2.54mm_Horizontal, symbol Connector_Generic:Conn_02x03_Row_Letter_Last
- added J10, J9: Conn_02x03_Odd_Even, Connector_PinHeader_2.54mm:PinHeader_2x03_P2.54mm_Vertical, symbol Connector_Generic:Conn_02x03_Odd_Even
Connections:
- net +BATT: now also J10.3 (Pin_3), J10.4 (Pin_4), J9.3 (Pin_3), J9.4 (Pin_4)
- net GND: now also J10.5 (Pin_5), J10.6 (Pin_6), J9.5 (Pin_5), J9.6 (Pin_6)
- net PWM1: now also J9.2 (Pin_2)
- net PWM2: now also J9.1 (Pin_1)
- net PWM3: now also J10.2 (Pin_2)
- net PWM4: now also J10.1 (Pin_1)
